File: 01_Hardware/PlantBuddy.kicad_pcb (KiCad board)
At the start: 4 copper layers, 35 x 87.7 mm, 68 parts, among them J1 SWD, Q1 AO3401, Q2 FS8205, Q3 FS8205, U1 CN301, U2 INA138, U3 LMC555xM, U4 XC6206P332MR, U5 BlueNRG-M1, U6 SHT20, U7 CN3063, U8 DW01+G, Y1 16MHz, Y2 32kHz

Commit message: PCB almost done
Parts:
- removed the Q3 at (138.6, 108.7)
- added Q2: FS8205, Package_TO_SOT_SMD:SOT-23-6, F.Cu at (75.9, 74.4)
- C18: value 2pF -> 2.2pF
- moved C26 115.0 mm to (61.2, 56.6), turned to 270 degrees
- moved Q1 113.2 mm to (57.6, 76.3), turned to 180 degrees
- moved R4 111.9 mm to (54.2, 63.9), turned to 270 degrees
- moved R3 110.8 mm to (51.0, 67.7), turned to 270 degrees
- moved C10 108.0 mm to (69.9, 57.8), turned to 90 degrees
- moved C18 106.1 mm to (65.8, 60.2), turned to 180 degrees
- moved C14 104.3 mm to (56.0, 64.3)
- moved C5 103.5 mm to (51.6, 59.1), turned to 90 degrees
- moved D1 101.7 mm to (57.1, 58.4), turned to 270 degrees
- moved R12 101.6 mm to (61.9, 63.5), turned to 90 degrees
- moved Y1 101.1 mm to (71.7, 61.5), turned to 90 degrees
- moved L3 99.9 mm to (62.8, 58.2), turned to 180 degrees
- moved C3 99.8 mm to (54.0, 56.4), turned to 180 degrees
- moved R1 98.9 mm to (53.4, 61.6), turned to 180 degrees
- moved C23 98.5 mm to (61.3, 58.6), turned to 90 degrees
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- renumbered Q2 to Q3
Connections:
- C1 pad 1: VCC -> /Vhum
- C19 pad 2: Net-(C18-Pad2) -> Net-(C18-Pad1)
- C20 pad 2: Net-(C18-Pad1) -> Net-(C18-Pad2)
- L1 pad 1: Net-(C18-Pad2) -> Net-(C18-Pad1)
- L2 pad 1: Net-(C18-Pad1) -> Net-(C18-Pad2)
- Q1 pad 3: VCC -> /Vhum
- Q3 pad 2: VCC -> Net-(Q3-Pad2)
- Q3 pad 5: Net-(Q2-Pad5) -> Net-(Q3-Pad2)
- Q3 pad 6: /IRR_EN -> Net-(Q3-Pad6)
- R8 pad 1: VCC -> /Vhum
- U3 pad 4: VCC -> /Vhum
- U3 pad 8: VCC -> /Vhum
- U5 pad 20: Net-(C18-Pad2) -> Net-(C18-Pad1)
- U5 pad 21: Net-(C18-Pad1) -> Net-(C18-Pad2)
- U5 pad 28: Net-(C16-Pad1) -> (no net)
Routing:
- net +3V3: track 0.00 -> 30.0 mm, vias 0 -> 8
- net +BATT: track 0.00 -> 30.0 mm, vias 0 -> 2
- net /THR: track 0.00 -> 24.8 mm
- net /Vhum: track 0.00 -> 18.9 mm, vias 0 -> 2
- net /fHumidity: track 0.00 -> 15.5 mm, vias 0 -> 2
- net VCC: track 0.00 -> 13.3 mm
- net /SCL: track 0.00 -> 12.5 mm
- net /~CHG_DONE: track 0.00 -> 11.8 mm, vias 0 -> 2
- net /~CHG_ON: track 0.00 -> 11.5 mm, vias 0 -> 2
- net Net-(BT1-Pad2): track 0.00 -> 10.5 mm, vias 0 -> 1
- net /SDA: track 0.00 -> 10.5 mm
- net /SXTAL0: track 0.00 -> 10.1 mm
- net /SXTAL1: track 0.00 -> 9.51 mm
- net Net-(Q3-Pad2): track 0.00 -> 8.77 mm
- net Net-(R1-Pad2): track 0.00 -> 8.01 mm
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- added copper zone on In2.Cu, net +3V3
- added copper zone on F.Cu, net -BATT
Other:
- net class Default: trace_width 0.25 -> 0.1524; via_dia 0.8 -> 0.55; via_drill 0.4 -> 0.3
- rule trace_min: 0.2 -> 0.15

Commit message: Initial Layout done
Parts:
- removed C16: 100nF, Capacitor_SMD:C_0603_1608Metric
- J1: moved to B.Cu
- SC1: footprint TestPoint:TestPoint_2Pads_Pitch5.08mm_Drill1.3mm -> PlantBuddy:SolarCell; moved to B.Cu
- moved C25 67.7 mm to (65.6, 78.3), turned to 180 degrees
- moved D3 63.8 mm to (65.6, 76.3)
- moved C8 63.7 mm to (59.1, 59.3)
- moved J1 63.3 mm to (65.7, 77.9), turned to 180 degrees
- moved C15 62.4 mm to (68.8, 76.2), turned to 270 degrees
- moved SC1 61.2 mm to (65.7, 75.7)
- moved R10 58.6 mm to (72.3, 57.4), turned to 0 degrees
- moved R11 56.6 mm to (74.7, 59.0), turned to 270 degrees
- moved R6 5.94 mm to (71.0, 70.8)
- moved R13 0.16 mm to (63.9, 69.9)
Connections:
- U5 pad 27: Net-(C16-Pad1) -> (no net)
Routing:
- net /VPanel: track 2.15 -> 50.8 mm, vias 0 -> 2
- net +BATT: track 30.0 -> 57.6 mm, vias 2 -> 3
- net /~LBO_ISR: track 0.00 -> 24.0 mm, vias 0 -> 2
- net /~HEN~: track 1.50 -> 19.2 mm, vias 0 -> 2
- net /IRR_EN: track 4.87 -> 21.3 mm, vias 0 -> 2
- net Net-(R10-Pad2): track 0.00 -> 15.3 mm
- net +3V3: track 30.0 -> 44.9 mm, vias 8 -> 12
- net /SWDIO: track 0.00 -> 14.4 mm, vias 0 -> 1
- net /SWCLK: track 0.00 -> 14.3 mm, vias 0 -> 1
- net -BATT: track 8.00 -> 17.5 mm, vias 151 -> 191
- net /ADC1: track 3.32 -> 12.3 mm, vias 0 -> 2
- net VCC: track 13.3 -> 18.9 mm
- net Net-(D3-Pad2): track 0.00 -> 2.98 mm, vias 0 -> 1
Other:
- board size 35 x 87.7 mm -> 35 x 87.3 mm
- net class CapacitiveProbe added: clearance 0.127, trace_width 0.1524, via_dia 0.55, via_drill 0.3

Commit message: Ordered PCB
Parts:
- added G***: LOGO, PlantBuddy:qr, B.Cu at (65.8, 64.6)
- C26: value 22pF -> 20pF
- R16: value 160R -> 1k
- R8: value Ra -> 330k
- R9: value Rb -> 330k
- moved D2 0.21 mm to (65.7, 69.9)
- turned R5 to 180 degrees
Connections:
- U2 pad 3: VCC -> /VPanel
- U2 pad 4: /VPanel -> VCC
Routing:
- net VCC: track 18.9 -> 17.0 mm
- net /VPanel: track 50.8 -> 50.2 mm
Other:
- board text added: "+"
- board text added: "-"
- board text added: "3V3"
- board text added: "CLK"
- board text added: "DIO"
- board text added: "GND"

Commit message: Evrika! We have an LED blinking! 🔥🎉💯
Parts:
- removed G***: LOGO, PlantBuddy:qr
- U6: value SHT20 -> SHT21
Connections:
- U5 pad 27: (no net) -> +3V3
Routing:
- net +3V3: track 44.9 -> 46.6 mm

Commit message: Revised PCB
Parts:
- removed C15, C24: 100nF, Capacitor_SMD:C_0603_1608Metric
- removed C17, C21, C25: 22uF, Capacitor_SMD:C_0603_1608Metric
- removed D3: B5819W, Diode_SMD:D_SOD-123
- removed Q3: FS8205, Package_TO_SOT_SMD:SOT-23-6
- removed R10, R11, R17: 120k, Resistor_SMD:R_0603_1608Metric
- removed R18: 160R, Resistor_SMD:R_0603_1608Metric
- removed R19, R7: 10k, Resistor_SMD:R_0603_1608Metric
- removed R4: 1M, Resistor_SMD:R_0603_1608Metric
- removed R5: 1R0, Resistor_SMD:R_0603_1608Metric
- removed R6: 470k, Resistor_SMD:R_0603_1608Metric
- removed SC1: Solar_Cell, PlantBuddy:SolarCell
- removed U2: INA138, Package_TO_SOT_SMD:SOT-23-5
- removed U4: XC6206P332MR, Package_TO_SOT_SMD:SOT-23
- removed U7: CN3063, Package_SO:SOP-8_3.9x4.9mm_P1.27mm
- removed U8: DW01+G, Package_TO_SOT_SMD:SOT-23-6
- added C16: 1uF, Capacitor_SMD:C_0402_1005Metric, F.Cu at (56.1, 66.0)
- added G***: LOGO, PlantBuddy:qr, B.Cu at (65.7, 62.7)
- added J2: Conn_I2C_SDA, TestPoint:TestPoint_Pad_D1.5mm, F.Cu at (71.0, 70.9)
- added J3: Conn_I2C_SCL, TestPoint:TestPoint_Pad_D1.5mm, F.Cu at (71.0, 73.6)
- added L4: 10uH, Inductor_SMD:L_0805_2012Metric, F.Cu at (58.8, 66.1)
- added SW1: PWR_SW, Button_Switch_SMD:SW_SPDT_CK-JS102011SAQN, F.Cu at (79.5, 64.4)
- added SW2: BLE_RST_SW, Button_Switch_SMD:SW_SPST_EVQP7C, F.Cu at (76.4, 75.2)
- BT1: footprint Battery:BatteryHolder_Keystone_1060_1x2032 -> PlantBuddy:BatteryHolder_LCSC_2032
- C1, C10, C12, C2, C7, C9: footprint Capacitor_SMD:C_0603_1608Metric -> Capacitor_SMD:C_0402_1005Metric
- C3, C5: value 2.2uF -> 100nF; footprint Capacitor_SMD:C_0603_1608Metric -> Capacitor_SMD:C_0402_1005Metric
- D1: value B5819W -> Y; footprint Diode_SMD:D_SOD-123 -> LED_SMD:LED_0603_1608Metric
- D2: value Status -> R
- J1: footprint Connector_JST:JST_SH_BM04B-SRSS-TB_1x04-1MP_P1.00mm_Vertical -> PlantBuddy:Debug_Connector
- Q2: value FS8205 -> AO3400A; footprint Package_TO_SOT_SMD:SOT-23-6 -> Package_TO_SOT_SMD:SOT-23
- R1: value 1M -> 10k; footprint Resistor_SMD:R_0603_1608Metric -> Resistor_SMD:R_0402_1005Metric
- R12, R13, R14, R15, R16, R2: footprint Resistor_SMD:R_0603_1608Metric -> Resistor_SMD:R_0402_1005Metric
- R3: value 1M -> 1k; footprint Resistor_SMD:R_0603_1608Metric -> Resistor_SMD:R_0402_1005Metric
- R8, R9: value 330k -> 10k; footprint Resistor_SMD:R_0805_2012Metric -> Resistor_SMD:R_0402_1005Metric
- U1: value CN301 -> OPT3001; footprint Package_TO_SOT_SMD:SOT-23-5 -> PlantBuddy:OPT3001DNPR
- U6: value SHT21 -> SHTC3; footprint Package_DFN_QFN:DFN-6-1EP_3x3mm_P1mm_EP1.5x2.4mm -> PlantBuddy:Sensirion_DFN-4-1EP_2x2mm_P1mm_EP0.7x1.6mm
- moved R1 27.4 mm to (78.7, 71.9)
- moved C3 20.6 mm to (70.5, 68.7), turned to 0 degrees
- moved D1 19.5 mm to (66.6, 75.5), turned to 90 degrees
- moved R3 18.5 mm to (68.0, 75.1), turned to 90 degrees
- moved U1 14.1 mm to (64.1, 70.4)
- moved R13 8.85 mm to (72.5, 67.9), turned to 0 degrees
- moved J1 8.74 mm to (65.8, 69.1)
- moved R16 7.84 mm to (63.5, 75.1)
- moved C5 7.35 mm to (56.1, 65.0), turned to 180 degrees
- moved R12 6.54 mm to (56.9, 59.2), turned to 0 degrees
- moved C9 6.21 mm to (56.9, 60.3)
- moved D2 5.65 mm to (64.9, 75.5), turned to 90 degrees
- moved Q2 4.44 mm to (75.2, 70.0)
- moved R14 4.09 mm to (66.7, 73.1), turned to 180 degrees
- moved R15 4.07 mm to (64.7, 73.1), turned to 0 degrees
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Connections:
- net /LED renamed /LEDR
- net /Vhum renamed Net-(C1-Pad1)
- net /~HEN~ renamed /~SOIL_EN~
- AE1 pad 2: -BATT -> GND
- BT1 pad 1: +BATT -> Net-(BT1-Pad1)
- C1 pad 2: -BATT -> GND
- C10 pad 1: +3V3 -> +BATT
- C10 pad 2: -BATT -> GND
- C11 pad 1: -BATT -> GND
- C12 pad 1: +3V3 -> +BATT
- C12 pad 2: -BATT -> GND
- C13 pad 1: -BATT -> GND
- C14 pad 1: -BATT -> GND
- C2 pad 2: -BATT -> GND
- C20 pad 1: -BATT -> GND
- C22 pad 1: -BATT -> GND
- C23 pad 1: -BATT -> GND
- C3 pad 2: -BATT -> GND
- C4 pad 2: -BATT -> GND
- C5 pad 1: +3V3 -> Net-(C16-Pad1)
- C5 pad 2: -BATT -> GND
- C6 pad 1: -BATT -> GND
- C7 pad 1: +3V3 -> +BATT
- C7 pad 2: -BATT -> GND
- C8 pad 1: -BATT -> GND
- C8 pad 2: +3V3 -> +BATT
- C9 pad 2: -BATT -> GND
- D1 pad 1: +BATT -> GND
- D1 pad 2: +3V3 -> Net-(D1-Pad2)
- D2 pad 1: -BATT -> GND
- J1 pad 1: Net-(D3-Pad2) -> +BATT
- J1 pad 4: -BATT -> GND
- L1 pad 2: -BATT -> GND
- Q1 pad 2: +3V3 -> +BATT
- Q2 pad 1: -BATT -> Net-(BT1-Pad1)
- Q2 pad 2: VCC -> GND
- Q2 pad 3: (no net) -> Net-(BT1-Pad2)
- R1 pad 1: -BATT -> +BATT
- R1 pad 2: Net-(R1-Pad2) -> /~BLE_RST
- R12 pad 1: +3V3 -> +BATT
- R13 pad 2: -BATT -> GND
- R14 pad 1: +3V3 -> +BATT
- R14 pad 2: /SDA -> /SCL
- R15 pad 1: +3V3 -> +BATT
- R15 pad 2: /SCL -> /SDA
- R2 pad 1: +3V3 -> +BATT
- R3 pad 1: Net-(R1-Pad2) -> Net-(D1-Pad2)
- R3 pad 2: +BATT -> /LEDY
- U1 pad 1: -BATT -> +BATT
- U1 pad 2: +BATT -> GND
- U1 pad 3: /~LBO_ISR -> GND
- U1 pad 4: Net-(R1-Pad2) -> /SCL
- U1 pad 5: (no net) -> /LUX_INT
- U3 pad 1: -BATT -> GND
- U5 pad 10: /~CHG_ON -> (no net)
- U5 pad 15: /ADC1 -> (no net)
- U5 pad 16: Net-(R10-Pad2) -> (no net)
- U5 pad 19: +3V3 -> +BATT
- U5 pad 24: +3V3 -> +BATT
- U5 pad 26: (no net) -> Net-(L4-Pad1)
- U5 pad 27: +3V3 -> Net-(C16-Pad1)
- U5 pad 3: /IRR_EN -> /LUX_INT
- U5 pad 31: -BATT -> GND
- U5 pad 33: -BATT -> GND
- U5 pad 6: +3V3 -> +BATT
- U5 pad 7: /~LBO_ISR -> /~BLE_RST
- U5 pad 9: /~CHG_DONE -> /LEDY
- U6 pad 1: /SDA -> +BATT
- U6 pad 2: -BATT -> /SCL
- U6 pad 3: (no net) -> /SDA
- U6 pad 4: (no net) -> GND
- U6 pad 5: +3V3 -> (no net)
- Y1 pad 2: -BATT -> GND
- Y1 pad 4: -BATT -> GND
Routing:
- net /VPanel: track 50.2 -> 0.00 mm, vias 2 -> 0
- net +3V3: track 46.6 -> 0.00 mm, vias 12 -> 0
- net Net-(BT1-Pad1): track 0.00 -> 31.9 mm, vias 0 -> 1
- net /~LBO_ISR: track 24.0 -> 0.00 mm, vias 2 -> 0
- net /IRR_EN: track 21.3 -> 0.00 mm, vias 2 -> 0
- net /~BLE_RST: track 0.00 -> 20.9 mm, vias 0 -> 2
- net -BATT: track 17.5 -> 0.00 mm, vias 191 -> 0
- net /SDA: track 10.5 -> 27.5 mm, vias 0 -> 4
- net VCC: track 17.0 -> 0.00 mm
- net +BATT: track 57.6 -> 40.9 mm, vias 3 -> 14
- net GND: track 0.00 -> 16.6 mm, vias 0 -> 178
- net Net-(R10-Pad2): track 15.3 -> 0.00 mm
- net /LEDR: track 2.63 -> 16.9 mm, vias 0 -> 2
- net /ADC1: track 12.3 -> 0.00 mm, vias 2 -> 0
- net /~CHG_DONE: track 12.0 -> 0.00 mm, vias 2 -> 0
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- added copper zone on In2.Cu, net +BATT
- added copper zone on F.Cu, net GND
- added copper zone on In1.Cu, net GND
- removed copper zone on In2.Cu, net +3V3
- removed copper zone on F.Cu, net -BATT
- removed copper zone on In1.Cu, net -BATT
Other:
- board text added: "OFF"
- board text added: "ON"
- board text added: "SCL"
- board text added: "SDA"
- board text added: "SYS RST"
- board text removed: "+"
- board text removed: "-"

Commit message: Ordered PCB version 2
Parts:
- added REF**: ToolingHole, PlantBuddy:ToolingHole, F.Cu at (65.7, 129.5)
- added REF**: ToolingHole, PlantBuddy:ToolingHole, F.Cu at (75.6, 49.8)
- added REF**: ToolingHole, PlantBuddy:ToolingHole, F.Cu at (55.8, 49.9)
- U1: footprint PlantBuddy:OPT3001DNPR -> Package_DFN_QFN:DFN-6-1EP_2x2mm_P0.65mm_EP1x1.6mm
Routing:
- net GND: track 16.6 -> 16.8 mm, vias 178 -> 179
