File: 01_Hardware/PlantBuddy.sch (KiCad schematic (older format))
At the start: 38 parts, among them J101 Debug, J102 NFC Antenna, J2 Conn_I2C_SDA, J3 Conn_I2C_SCL, Q2 AO3400A, U1 OPT3001, U101 nRF52832-QFxx, U6 SHTC3, Y1 32MHz, Y2 32kHz

Commit message: HW: Rev 4.1 => Changed ALS from OPT3001 to LTR-303
Parts:
- removed U1: OPT3001, Package_DFN_QFN:DFN-6-1EP_2x2mm_P0.65mm_EP1x1.6mm, symbol PlantBuddy:OPT3001
- added U102: LTR-303ALS-01, OptoDevice:Lite-On_LTR-303ALS-01, symbol Sensor_Optical:LTR-303ALS-01
Connections:
- wire segments 95 -> 96
Other:
- note added: "0 to 65535 Lux Light sensor"
- note removed: "0 to 83865 Lux Light sensor"
- moved on the sheet: C3
Changed lines of the file:
@@
 L PlantBuddy-rescue:+BATT-power #PWR010
 U 1 1 5F85BEB5
-P 1400 6450
-F 0 "#PWR010" H 1400 6300 50  0001 C CNN
-F 1 "+BATT" H 1275 6575 50  0000 C CNN
-F 2 "" H 1400 6450 50  0001 C CNN
-F 3 "" H 1400 6450 50  0001 C CNN
-	1    1400 6450
+P 1400 6350
+F 0 "#PWR010" H 1400 6200 50  0001 C CNN
+F 1 "+BATT" H 1225 6625 50  0000 C CNN
+F 2 "" H 1400 6350 50  0001 C CNN
+F 3 "" H 1400 6350 50  0001 C CNN
+	1    1400 6350
 	-1   0    0    -1
 $EndComp
-Text Label 2075 6750 2    50   ~ 0
+Text Label 2075 6650 2    50   ~ 0
 SDA
-Text Label 2075 6650 2    50   ~ 0
-SCL
 $Comp
 L PlantBuddy-rescue:GND-power #PWR0101
@@
 	-1   0    0    -1
 $EndComp
-Text Label 2150 6950 2    50   ~ 0
+Text Label 650  6750 0    50   ~ 0
 LUX_INT
 Wire Wire Line
-	2150 6950 1800 6950
+	650  6750 1000 6750
 $Comp
 L PlantBuddy-rescue:GND-power #PWR026
@@
 Wire Wire Line
 	1800 6650 2075 6650
-Wire Wire Line
-	1800 6750 2075 6750
 Wire Wire Line
 	2475 5125 2475 5225
@@
 	2375 5550 3075 5550
 Wire Wire Line
-	1400 7150 1000 7150
-Wire Wire Line
-	1000 6650 1000 6450
-Wire Wire Line
-	1000 6450 1400 6450
-Wire Wire Line
 	3725 7300 3550 7300
 Wire Wire Line
@@
 Text Notes 2825 7675 0    50   ~ 0
 Reverse-voltage protection
-Wire Wire Line
-	1000 6850 1000 6950
-Connection ~ 1400 6450
-Connection ~ 1000 6950
-Wire Wire Line
-	1000 6950 1000 7150
-Connection ~ 1400 7150
 Text Notes 9825 5225 0    50   ~ 0
 Yellow status LED => short blinks\nto notify user of different actions
@@
 L PlantBuddy-rescue:C_Small-Device C3
 U 1 1 5FC58638
-P 1000 6750
-F 0 "C3" H 850 6850 50  0000 L CNN
-F 1 "100nF" H 700 6700 50  0000 L CNN
-F 2 "Capacitor_SMD:C_0402_1005Metric" H 1000 6750 50  0001 C CNN
-F 3 "~" H 1000 6750 50  0001 C CNN
-F 4 "C1525" H 1000 6750 50  0001 C CNN "LCSC"
-	1    1000 6750
+P 550 6750
+F 0 "C3" H 600 6900 50  0000 L CNN
+F 1 "100nF" H 600 6625 50  0000 L CNN
+F 2 "Capacitor_SMD:C_0402_1005Metric" H 550 6750 50  0001 C CNN
+F 3 "~" H 550 6750 50  0001 C CNN
+F 4 "C1525" H 550 6750 50  0001 C CNN "LCSC"
+	1    550  6750
 	1    0    0    -1
 $EndComp
@@
 $EndComp
 $Comp
-L PlantBuddy:OPT3001 U1
-U 1 1 5FD09708
-P 1400 7200
-F 0 "U1" H 1400 8221 50  0000 C CNN
-F 1 "OPT3001" H 1600 7900 50  0000 C CNN
-F 2 "Package_DFN_QFN:DFN-6-1EP_2x2mm_P0.65mm_EP1x1.6mm" H 1400 7200 50  0001 C CNN
-F 3 "https://www.ti.com/lit/ds/symlink/opt3001.pdf" H 1400 7200 50  0001 C CNN
-F 4 "C90462" H 1600 7275 50  0001 C CNN "LCSC"
-	1    1400 7200
-	1    0    0    -1
-$EndComp
-$Comp
 L PlantBuddy-rescue:LED_Small-Device D1
 U 1 1 5FC270B5
@@
 Wire Wire Line
 	9825 875  10100 875
-Text Notes 1950 7500 2    50   ~ 0
-0 to 83865 Lux Light sensor
+Text Notes 1850 7500 2    50   ~ 0
+0 to 65535 Lux Light sensor
 $Comp
 L PlantBuddy-rescue:C_Small-Device C11
@@
 	1    0    0    -1
 $EndComp
-Wire Bus Line
-	2175 5325 2625 5325
-Wire Bus Line
-	2175 5325 2175 6650
 Text Label 9825 1175 0    50   ~ 0
 UART_Rx
@@
 	1    0    0    -1
 $EndComp
+Connection ~ 1400 6350
+$Comp
+L Sensor_Optical:LTR-303ALS-01 U102
+U 1 1 611AA492
+P 1400 6750
+F 0 "U102" H 1400 7331 50  0000 C CNN
+F 1 "LTR-303ALS-01" H 1050 6350 50  0000 C CNN
+F 2 "OptoDevice:Lite-On_LTR-303ALS-01" H 1400 7200 50  0001 C CNN
+F 3 "http://optoelectronics.liteon.com/upload/download/DS86-2013-0004/LTR-303ALS-01_DS_V1.pdf" H 1100 7100 50  0001 C CNN
+	1    1400 6750
+	-1   0    0    -1
+$EndComp
+Wire Wire Line
+	550  6350 550  6650
+Wire Wire Line
+	550  6350 1400 6350
+Wire Wire Line
+	1400 7150 550  7150
+Wire Wire Line
+	550  6850 550  7150
+Connection ~ 1400 7150
+Text Label 2075 6750 2    50   ~ 0
+SCL
+Wire Wire Line
+	2075 6750 2025 6750
+Wire Wire Line
+	2025 6750 2025 6850
+Wire Wire Line
+	2025 6850 1800 6850
+Wire Bus Line
+	2175 5325 2625 5325
+Wire Bus Line
+	2175 5325 2175 6650
 $EndSCHEMATC

Commit message: Started PCB improvements & added SVGs and interactive BOM.
Parts:
- removed Q2: AO3400A, Package_TO_SOT_SMD:SOT-23, symbol PlantBuddy-rescue:Q_NMOS_GSD-Device
- added Q101: AO3401A, Package_TO_SOT_SMD:SOT-23, symbol Transistor_FET:AO3401A
- BT1: footprint PlantBuddy:BatteryHolder_LCSC_2032 -> PlantBuddy:BAT-HLD-001; LCSC C70377 -> (none)
- C15: value 4.7uF -> 1uF; LCSC C23733 -> C52923
Other:
- note added: "TODO: Consider micro-speaker with low-cost low-power driver"
- note added: "TODO: Current debug connector is THT and non-standard.\nMake it SMD and standard."
- note added: "TODO: Do we really need NFC?"
- moved on the sheet: R4
Changed lines of the file:
@@
 Wire Wire Line
 	2375 5550 3075 5550
-Wire Wire Line
-	3725 7300 3550 7300
-Wire Wire Line
-	2875 7300 3150 7300
 Text Notes 2825 7675 0    50   ~ 0
 Reverse-voltage protection
 Text Notes 9825 5225 0    50   ~ 0
 Yellow status LED => short blinks\nto notify user of different actions
-$Comp
-L PlantBuddy-rescue:Q_NMOS_GSD-Device Q2
-U 1 1 5FC7486C
-P 3350 7200
-F 0 "Q2" V 3599 7200 50  0000 C CNN
-F 1 "AO3400A" V 3690 7200 50  0000 C CNN
-F 2 "Package_TO_SOT_SMD:SOT-23" H 3550 7300 50  0001 C CNN
-F 3 "https://datasheet.lcsc.com/szlcsc/1811081213_Alpha-Omega-Semicon-AO3400A_C20917.pdf" H 3350 7200 50  0001 C CNN
-F 4 "C20917" V 3350 7200 50  0001 C CNN "LCSC"
-	1    3350 7200
-	0    -1   1    0
-$EndComp
 $Comp
 L PlantBuddy-rescue:Conn_01x01-Connector_Generic J3
@@
 $EndComp
 $Comp
-L PlantBuddy-rescue:Battery_Cell-Device BT1
-U 1 1 5FC5077F
-P 2875 7100
-F 0 "BT1" H 2993 7196 50  0000 L CNN
-F 1 "Li+" H 2993 7105 50  0000 L CNN
-F 2 "PlantBuddy:BatteryHolder_LCSC_2032" V 2875 7160 50  0001 C CNN
-F 3 "~" V 2875 7160 50  0001 C CNN
-F 4 "C70377" H 2875 7100 50  0001 C CNN "LCSC"
-F 5 "CR2032-BS-6-1" H 2875 7100 50  0001 C CNN "MFR"
-	1    2875 7100
-	1    0    0    -1
-$EndComp
-$Comp
 L PlantBuddy-rescue:R_Small-Device R15
 U 1 1 5F7AB23C
@@
 L PlantBuddy-rescue:R_Small-Device R4
 U 1 1 6047E951
-P 3350 6900
-F 0 "R4" H 3200 6950 50  0000 L CNN
-F 1 "10k" H 3175 6875 50  0000 L CNN
-F 2 "Resistor_SMD:R_0402_1005Metric" H 3350 6900 50  0001 C CNN
-F 3 "~" H 3350 6900 50  0001 C CNN
-F 4 "C25744" H 3350 6900 50  0001 C CNN "LCSC"
-	1    3350 6900
+P 3325 7200
+F 0 "R4" H 3175 7250 50  0000 L CNN
+F 1 "10k" H 3150 7175 50  0000 L CNN
+F 2 "Resistor_SMD:R_0402_1005Metric" H 3325 7200 50  0001 C CNN
+F 3 "~" H 3325 7200 50  0001 C CNN
+F 4 "C25744" H 3325 7200 50  0001 C CNN "LCSC"
+	1    3325 7200
 	-1   0    0    -1
 $EndComp
-Wire Wire Line
-	2875 6800 3350 6800
-Connection ~ 3350 6800
-Wire Wire Line
-	3350 6800 3725 6800
 Wire Wire Line
 	2875 6900 2875 6800
@@
 $EndComp
 Wire Wire Line
-	7375 3175 7000 3175
+	7375 3075 7000 3075
 Wire Wire Line
 	7375 3675 7000 3675
@@
 $EndComp
 Wire Wire Line
-	7375 3075 7000 3075
+	7375 3175 7000 3175
+Text Label 7375 3075 2    50   ~ 0
+LEDY
 Text Label 7375 3175 2    50   ~ 0
-LEDY
-Text Label 7375 3075 2    50   ~ 0
 LUX_INT
 NoConn ~ 5700 1475
@@
 P 8425 1100
 F 0 "C15" H 8517 1146 50  0000 L CNN
-F 1 "4.7uF" H 8517 1055 50  0000 L CNN
+F 1 "1uF" H 8517 1055 50  0000 L CNN
 F 2 "Capacitor_SMD:C_0402_1005Metric" H 8425 1100 50  0001 C CNN
-F 3 "https://datasheet.lcsc.com/szlcsc/Samsung-Electro-Mechanics-CL05A475MP5NRNC_C23733.pdf" H 8425 1100 50  0001 C CNN
-F 4 "C23733" H 8425 1100 50  0001 C CNN "LCSC"
+F 3 "~" H 8425 1100 50  0001 C CNN
+F 4 "C52923" H 8425 1100 50  0001 C CNN "LCSC"
 	1    8425 1100
 	1    0    0    -1
@@
 Wire Wire Line
 	2025 6850 1800 6850
+Text Notes 9825 1500 0    50   ~ 0
+TODO: Current debug connector is THT and non-standard.\nMake it SMD and standard.
+Text Notes 9825 5500 0    50   ~ 0
+TODO: Consider micro-speaker with low-cost low-power driver
+$Comp
+L PlantBuddy-rescue:Battery_Cell-Device BT1
+U 1 1 5FC5077F
+P 2875 7100
+F 0 "BT1" H 2993 7196 50  0000 L CNN
+F 1 "Li+" H 2993 7105 50  0000 L CNN
+F 2 "PlantBuddy:BAT-HLD-001" V 2875 7160 50  0001 C CNN
+F 3 "~" V 2875 7160 50  0001 C CNN
+F 4 "" H 2875 7100 50  0001 C CNN "LCSC"
+F 5 "CR2032-BS-6-1" H 2875 7100 50  0001 C CNN "MFR"
+	1    2875 7100
+	1    0    0    -1
+$EndComp
+$Comp
+L Transistor_FET:AO3401A Q101
+U 1 1 6134A6DD
+P 3325 6900
+F 0 "Q101" V 3667 6900 50  0000 C CNN
+F 1 "AO3401A" V 3576 6900 50  0000 C CNN
+F 2 "Package_TO_SOT_SMD:SOT-23" H 3525 6825 50  0001 L CIN
+F 3 "http://www.aosmd.com/pdfs/datasheet/AO3401A.pdf" H 3325 6900 50  0001 L CNN
+	1    3325 6900
+	0    -1   -1   0
+$EndComp
+Wire Wire Line
+	3125 6800 2875 6800
+Wire Wire Line
+	3525 6800 3725 6800
+Wire Wire Line
+	2875 7300 3325 7300
+Wire Wire Line
+	3325 7300 3725 7300
+Connection ~ 3325 7300
 Wire Bus Line
 	2175 5325 2625 5325
 Wire Bus Line
 	2175 5325 2175 6650
+Text Notes 7875 2850 0    50   ~ 0
+TODO: Do we really need NFC?
 $EndSCHEMATC
